Commit message: update

File: urdf/husky_with_Lidar.urdf.xacro (robot description, xacro)
@@ -24,5 +24,5 @@
   </joint>
   <xacro:include filename="$(find velodyne_description)/urdf/VLP-16.urdf.xacro"/>
-  <xacro:VLP-16 parent="base_link" name="velodyne" topic="/velodyne_points" hz="10" samples="440" gpu="${gpu}">
+  <xacro:VLP-16 parent="base_link" name="velodyne" topic="/velodyne_points" hz="10" samples="4400" gpu="${gpu}">
     <origin xyz="0 -3 0.7" rpy="0 0.5 0" />
   </xacro:VLP-16>

File: urdf/realsense.urdf.xacro (robot description, xacro)
@@ -11,5 +11,5 @@
     <parent link="front_realsense"/>
     <child link="front_realsense_gazebo"/>
-    <origin xyz="0.0 0 0.5" rpy="-1.5707963267948966 0 -1.5707963267948966"/>
+    <origin xyz="0.0 0 -0.5" rpy="-1.5707963267948966 0 -1.5707963267948966"/>
     <!--origin xyz="0.0 0 0.5" rpy="-2.094395102 0 -1.5707963267948966"/-->
   </joint>
