Commit message: RVIZ visualization and LiDAR

File: amiga_description/urdf/amiga.urdf.xacro (robot description, xacro)
@@ -8,4 +8,28 @@
   <!-- Load amiga description -->
   <!-- <xacro:amiga prefix="$(arg prefix)" /> -->
+  <xacro:arg name="gpu" default="true"/>
+  <xacro:property name="gpu" value="$(arg gpu)" />
+  <xacro:if value="$(arg lidar)">
+    <link name="velodyne_link">
+    <visual>
+      <!-- Specify visual properties for the LiDAR -->
+    </visual>
+    <collision>
+      <!-- Specify collision properties for the LiDAR -->
+    </collision>
+    <inertial>
+      <!-- Specify inertial properties for the LiDAR -->
+    </inertial>
+  </link>
+  <joint name="velodyne_joint" type="fixed">
+    <origin xyz="0 0 0.0" rpy="0 0 0"/>
+    <parent link="base_link"/>
+    <child link="velodyne_link"/>
+  </joint>
+    <xacro:include filename="$(find velodyne_description)/urdf/VLP-16.urdf.xacro" />
+    <xacro:VLP-16 parent="base_link" name="velodyne" topic="/velodyne_points" hz="10" samples="8000" gpu="${gpu}">
+      <origin xyz="1 0 1.5" rpy="0 0.7 0" />
+    </xacro:VLP-16>
+  </xacro:if>
   <xacro:if value="$(arg is_sim)">
     <gazebo>

File: amiga_description/urdf/farm-ng.urdf.xacro (robot description, xacro)
@@ -1,4 +1,5 @@
 <?xml version="1.0"?>
 <robot xmlns:xacro="http://www.ros.org/wiki/xacro" name="amiga">
+<xacro:arg name="is_sim" default="true" />
 <!-- <robot xmlns:xacro="http://ros.org/wiki/xacro"> -->
 <!-- <xacro:include filename="$(find amiga_description)/urdf/wheel.urdf.xacro" /> -->
@@ -19,13 +20,14 @@
 <link name="inertial_link">
     <inertial>
-        <!-- <origin xyz="0.0 0.0 0.22" rpy="0.0 0.0 0.0"/>
-        <mass value="158.0"/> -->
-        <!-- <inertia ixx="294.935" ixy="0.0" ixz="0.0"
-                 iyy="380.351" iyz="0.0"
-                 izz="167.104"/> -->
-        <mass value="46.034" />
+        <origin xyz="0.0 0.0 0.22" rpy="0.0 0.0 0.0"/>
+        <mass value="158.0"/>
+        <inertia ixx="43.75" ixy="0.0" ixz="0.0"
+                 iyy="32.74" iyz="0.0"
+                 izz="50.15"/>
+        </inertial>
+        <!-- <mass value="46.034" />
         <origin xyz="-0.00065 -0.0 0.22" />
         <inertia ixx="0.6022" ixy="-0.02364" ixz="-0.1197" iyy="1.7386" iyz="-0.001544" izz="2.0296" />
-    </inertial>
+    </inertial> -->
   </link>
   <joint name="inertial_joint" type="fixed">
@@ -215,11 +217,11 @@
         </collision>
     </link>
-    <gazebo reference="tire_${name}_link">
-      <mu1 value="1.0"/>
+    <!-- <gazebo reference="tire_${name}_link">
+      <mu1 value=".5"/>
       <mu2 value="0.5"/>
       <kp value="1000000.0" />
       <kd value="1.0" />
       <fdir1 value="1 0 0"/>
-    </gazebo>
+    </gazebo> -->
     <joint name="tire_${name}_joint" type="continuous">
         <origin xyz="${x} ${y} ${z}" rpy="0 0.0 0.0"/>
@@ -274,4 +276,15 @@
     <axis xyz="0.0 0.0 0.0"/>
 </joint>
+<!-- <link name="velodyne_link">
+</link>
+<joint name="velodyne_joint" type="fixed">
+    <origin xyz="0 0 0.0" rpy="0 0 0" />
+    <parent link="base_link" />
+    <child link="velodyne_link" />
+</joint> -->
+<!--<xacro:include filename="$(find amiga_description)/urdf/VLP-16.urdf.xacro" />
+<xacro:VLP-16 parent="base_link" name="velodyne" topic="/velodyne_points" hz="10" samples="8000" gpu="true">
+    <origin xyz="1 0 1.5" rpy="0 0.7 0" />
+</xacro:VLP-16> -->
 <!-- </xacro:macro> -->
 <ros2_control name="GazeboSystem" type="system">

Commit message: update ros2 humble

File: amiga_description/urdf/amiga.urdf.xacro (robot description, xacro)
@@ -11,22 +11,6 @@
   <xacro:property name="gpu" value="$(arg gpu)" />
   <xacro:if value="$(arg lidar)">
-    <link name="velodyne_link">
-    <visual>
-      <!-- Specify visual properties for the LiDAR -->
-    </visual>
-    <collision>
-      <!-- Specify collision properties for the LiDAR -->
-    </collision>
-    <inertial>
-      <!-- Specify inertial properties for the LiDAR -->
-    </inertial>
-  </link>
-  <joint name="velodyne_joint" type="fixed">
-    <origin xyz="0 0 0.0" rpy="0 0 0"/>
-    <parent link="base_link"/>
-    <child link="velodyne_link"/>
-  </joint>
     <xacro:include filename="$(find velodyne_description)/urdf/VLP-16.urdf.xacro" />
-    <xacro:VLP-16 parent="base_link" name="velodyne" topic="/velodyne_points" hz="10" samples="8000" gpu="${gpu}">
+    <xacro:VLP-16 parent="base_link" name="velodyne" topic="/velodyne_points" hz="10" samples="4000" gpu="${gpu}">
       <origin xyz="1 0 1.5" rpy="0 0.7 0" />
     </xacro:VLP-16>
